File: Hardware/A-NET/A-NET.kicad_pcb (KiCad board)
At the start: 2 copper layers, 100 x 60 mm, 101 parts, among them IC1 74AHC1G125, J1 BAT, J2 USB_C_Receptacle_USB2.0_16P, J3 Digital/PWM, J4 Power, J5 Analog, J6 Digital/PWM, SW1 SW_MEC_5E, SW2 SW_MEC_5E, U1 TPS563252DRLR, U2 ESP32-S3-WROOM-1, U3 AMS1117-3.3, U4 RESET, X1 RB1-125BAG1A, Y1 25MHz

Commit message: Add files via upload
Parts:
- removed the C10 at (117.2, 96.8)
- removed the C11 at (118.8, 96.8)
- removed the C8 at (114.0, 97.8)
- removed the C9 at (114.0, 96.3)
- removed D10: LEDUSB, LED_SMD:LED_0603_1608Metric_Pad1.05x0.95mm_HandSolder
- removed the R10 at (120.4, 96.7)
- removed U3: AMS1117-3.3, Package_TO_SOT_SMD:SOT-223-3_TabPin2
- C4: renamed from C6; value 33p -> 56p
- D7: renamed from D11; moved to F.Cu
- D8: renamed from D13; moved to F.Cu
- D9: renamed from D14; moved to F.Cu
- IC1: footprint NSARCHI:74AHC1G125 -> anetLib:74AHC1G125
- R2: renamed from R5; value 47K -> 32K
- R3: renamed from R6; value 30K -> 10K
- SJ1, SJ2, SJ3: footprint NSARCHI:SJ -> anetLib:Jumper
- U$1: footprint NSARCHI:W5500 -> anetLib:W5500
- U1: footprint NSARCHI:SOT6_DRL_TEX-L -> anetLib:SOT6_DRL_TEX-L
- moved D7 24.0 mm to (154.7, 120.4)
- moved SW1 23.4 mm to (110.5, 125.1)
- moved D9 20.5 mm to (156.3, 120.3)
- moved C7 19.3 mm to (104.6, 126.9), turned to -90 degrees
- moved C11 17.7 mm to (112.0, 124.6)
- moved R10 17.2 mm to (108.8, 124.6), turned to 180 degrees
- moved D8 17.1 mm to (157.8, 120.3)
- moved R7 17.1 mm to (105.5, 124.6), turned to 0 degrees
- moved C10 16.3 mm to (118.6, 79.0), turned to 0 degrees
- moved FB2 14.3 mm to (169.1, 119.4), turned to 180 degrees
- moved R13 13.2 mm to (157.8, 120.3)
- moved R14 13.1 mm to (156.3, 120.3)
- moved R12 13.0 mm to (154.7, 120.4)
- moved C9 11.2 mm to (119.4, 94.5), turned to 0 degrees
- moved SW2 11.0 mm to (120.4, 125.2)
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- renumbered C7 to C10, C29 to C11, C28 to C12, C21 to C14, C23 to C15, C22 to C16, C24 to C17, C25 to C19, C26 to C21, C16 to C25, C17 to C26, C18 to C27, C19 to C28, C20 to C29, C13 to C33, C15 to C34, C12 to C35, C14 to C37, C27 to C42, C4 to C5, C5 to C6, C30 to C7, C31 to C8, C32 to C9, D7 to D3, D8 to D4, D9 to D5, J4 to J3, J5 to J4, J3 to J5, R2 to R1, R32 to R10, R31 to R11, R26 to R12, R28 to R13, R29 to R14, R22 to R15, R20 to R16, R21 to R18, R24 to R19, R25 to R21, R14 to R23, R15 to R25, R16 to R26, R17 to R27, R23 to R32, R11 to R39, R3 to R4, R18 to R40, R12 to R41, R19 to R42, R13 to R43, R30 to R46, R4 to R5, R1 to R6, R33 to R7, SW2 to SW1, SW1 to SW2, U4 to U6
Connections:
- net /Archi/GP07 renamed /Ethernet/RESET
- net /Archi/GP08 renamed /Ethernet/INTN
- net /Archi/GP09 renamed /Ethernet/CS
- net /Archi/GP10 renamed /Ethernet/SCK
- net /Archi/GP11 renamed /Ethernet/MOSI
- net /Archi/GP12 renamed /Archi/MISO
- net /Archi/GP13 renamed /Archi/CS1
- net /Archi/GP14 renamed /Archi/READY
- net /Archi/GP15 renamed /MCU-WiFi/GPIO0
- C10 pad 1: Vout -> VBAT
- C19 pad 2: AGND -> GND
- C4 pad 2: Vout -> +3V3
- C5 pad 1: Vout -> +3V3
- C6 pad 1: Vout -> +3V3
- C8 pad 1: +3V3USB -> +3V3
- C9 pad 1: +3V3USB -> +3V3
- D3 pad 1: Vout -> +3V3
- D4 pad 2: Vout -> +3V3
- D6 pad 1: Vout -> VBAT
- L1 pad 2: Vout -> +3V3
- R10 pad 2: +3V3USB -> +3V3
- R11 pad 2: +3V3USB -> +3V3
- R4 pad 2: Vout -> +3V3
- R5 pad 2: Vout -> +3V3
- R6 pad 1: Vout -> +3V3
- R7 pad 2: +3V3USB -> +3V3
- U$1 pad 1: /Ethernet/TX- -> Net-(U$1-TXN)
- U$1 pad 2: /Ethernet/TX+ -> Net-(U$1-TXP)
- U$1 pad 5: /Ethernet/RX- -> Net-(U$1-RXN)
- U$1 pad 6: /Ethernet/RX+ -> Net-(U$1-RXP)
- U2 pad 2: +3V3USB -> +3V3
- Y1 pad 3: (no net) -> Net-(U$1-XI/CLKIN)
- Y1 pad 4: (no net) -> Net-(U$1-XO)
Routing:
- net +3V3: track 122.2 -> 221.6 mm, vias 8 -> 17
- net Vout: track 56.2 -> 0.00 mm, vias 6 -> 0
- net /Archi/MISO: track 0.00 -> 54.3 mm, vias 0 -> 2
- net /Ethernet/MOSI: track 1.84 -> 52.8 mm, vias 1 -> 2
- net /Ethernet/SCK: track 2.31 -> 52.5 mm, vias 1 -> 2
- net /Ethernet/LINKLED: track 19.5 -> 55.7 mm
- net /Archi/CS1: track 0.00 -> 33.3 mm, vias 0 -> 1
- net /Ethernet/RESET: track 4.74 -> 37.2 mm, vias 1 -> 2
- net /Ethernet/ACTLED: track 20.4 -> 51.6 mm
- net GND: track 71.3 -> 40.2 mm, vias 43 -> 40
- net +3V3USB: track 27.6 -> 0.00 mm, vias 4 -> 0
- net /Ethernet/CS: track 16.6 -> 38.7 mm
- net /Archi/READY: track 0.00 -> 21.1 mm
- net /MCU-WiFi/GPIO0: track 13.8 -> 34.7 mm
- net /Ethernet/INTN: track 19.4 -> 37.7 mm
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- added copper zone on B.Cu, net +3V3
- removed copper zone on B.Cu, net +3V3USB
- removed copper zone on B.Cu, net Vout
