File: Hardware/A-NET/Archi.kicad_sch (KiCad schematic)
At the start: 7 parts, among them J3 Digital/PWM, J4 Power, J5 Analog, J6 Digital/PWM, U4 RESET

Commit message: add digikey | add POE
Parts:
- R46: renamed from R30; PartNumber RC0603FR-0710KL -> RCS060310K0JNEA; PurchaseLink https://www.digikey.com/en/products/detail/yageo/RC0603FR-0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 -> https://www.digikey.de/en/products/detail/vishay-dale/RCS06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
- renumbered C27 to C42, J4 to J3, J5 to J4, J3 to J5, U4 to U6
Other:
- note added: "VOUT 3V3"
- note removed: "MULTIPLEXOR: - S0 (GP06) - S1 (GP07) - S2 (GP08)"
- moved on the sheet: J4
