File: Hardware/A-NET/Ethernet.kicad_sch (KiCad schematic)
At the start: 45 parts, among them IC1 74AHC1G125, X1 RB1-125BAG1A, Y1 25MHz

Commit message: add digikey | add POE
Parts:
- removed X1: RB1-125BAG1A, NSARCHI:RB1-125BAG1A, symbol ArchiBot-eagle-import:RJ45J0026D21BNL
- added C13: 10uF/50V, CAP-1808, symbol A-NET-altium-import:root_1_CAP-1808
- added C18: 1uF, 50V, CAP-0805, symbol A-NET-altium-import:root_1_CAP-0805
- added C20: 47pF,100V, CAP-0805, symbol A-NET-altium-import:root_1_CAP-0805
- added C22: 0.1uF/50V, CAP-0805, symbol A-NET-altium-import:root_1_CAP-0805
- added C23: 22uF,10V, C3216TT(A), symbol A-NET-altium-import:root_0_TANTAL_CASE A(3216)
- added C24: 1uF/50V, CAP-0805, symbol A-NET-altium-import:root_2_CAP-0805
- added C30: 10uF,10V, C6032TT(C), symbol A-NET-altium-import:root_0_TANTAL_CASE A(3216)
- added C31: 47uF,10V, C3216TT(A), symbol A-NET-altium-import:root_0_TANTAL_CASE A(3216)
- added C32: 0.33uF,50V, CAP-0603, symbol A-NET-altium-import:root_1_CAP-0603
- added C36: 330uF,6V, C3216TT(A), symbol A-NET-altium-import:root_0_TANTAL_CASE A(3216)
- added C38: 0.1uF,50V, CAP-0603, symbol A-NET-altium-import:root_1_CAP-0603
- added C39: 1uF,16V, CAP-0603, symbol A-NET-altium-import:root_1_CAP-0603
- added C40: 10uF/16V, CAP-1808, symbol A-NET-altium-import:root_3_CAP-1808
- added C41: 470uF/16V, CAP-8.3EC, symbol A-NET-altium-import:root_0_AL-CAP-D 8.0mm_SMD
- added D10: SMAJ12, DO-214AC/SMA, symbol A-NET-altium-import:root_1_DIODE-Shottky (SOD-323)
- added D11: NC/SMAJ150A, DO-214AC/SMA, symbol A-NET-altium-import:root_1_DIODE-Shottky (SOD-323)
- added D12: BAV19, SOD-123(1-C,2-A), symbol A-NET-altium-import:root_2_DIODE-BAT60A
- added D13: RBR5L40A, DO-214AB/SMC, symbol A-NET-altium-import:root_0_DIODE-Shottky (SOD-323)
- added L2: SM13117EL, SM13117EL, symbol A-NET-altium-import:root_0_SM13117EL
- added L3: 1uH, 2A, IND-0805, symbol A-NET-altium-import:root_0_IND-0805
- added Q1: Q-2N7002, SOT23-3L, symbol A-NET-altium-import:root_3_Q-2N7002
- added R17: 24.9K, Resistor_SMD:R_0603_1608Metric, symbol ArchiBot-eagle-import:RESISTOR_0603_NOOUT
- added R20: 15K, Resistor_SMD:R_0603_1608Metric, symbol ArchiBot-eagle-import:RESISTOR_0603_NOOUT
- added R22: 51K, Resistor_SMD:R_0603_1608Metric, symbol ArchiBot-eagle-import:RESISTOR_0603_NOOUT
- added R24: 1M, Resistor_SMD:R_0603_1608Metric, symbol ArchiBot-eagle-import:RESISTOR_0603_NOOUT
- added R28: 0R, Resistor_SMD:R_0603_1608Metric, symbol ArchiBot-eagle-import:RESISTOR_0603_NOOUT
- added R29: 680K, Resistor_SMD:R_0603_1608Metric, symbol ArchiBot-eagle-import:RESISTOR_0603_NOOUT
- added R30, R31, R33, R34: 3.3R, Resistor_SMD:R_0603_1608Metric, symbol ArchiBot-eagle-import:RESISTOR_0603_NOOUT
- added R35: 5.1R, Resistor_SMD:R_0603_1608Metric, symbol ArchiBot-eagle-import:RESISTOR_0603_NOOUT
- added R36: 100R, Resistor_SMD:R_0603_1608Metric, symbol ArchiBot-eagle-import:RESISTOR_0603_NOOUT
- added R37: 75, Resistor_SMD:R_0603_1608Metric, symbol ArchiBot-eagle-import:RESISTOR_0603_NOOUT
- added R38: 1K, Resistor_SMD:R_0603_1608Metric, symbol ArchiBot-eagle-import:RESISTOR_0603_NOOUT
- added R44, R45: 30K, Resistor_SMD:R_0603_1608Metric, symbol ArchiBot-eagle-import:RESISTOR_0603_NOOUT
- added U3: DPA423-PN, DIP-08, symbol A-NET-altium-import:root_0_DPA423
- added U4: PC357, PC357, symbol A-NET-altium-import:root_0_PC357
- added U5: TL431ID, SOT23-3L, symbol A-NET-altium-import:root_2_TL431IDBZT
- added X1: 7499210121A, NSARCHI:RB1-125BAG1A, symbol archi:RJ45POE-1-2250024-1
- C14: renamed from C21; PartNumber (none) -> CC0402JRNPO7BN220; PurchaseLink (none) -> https://www.digikey.de/en/products/detail/yageo/CC0402JRNPO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
- C15: renamed from C23; PartNumber (none) -> CL10A106MQ8NNNC; PurchaseLink (none) -> https://www.digikey.de/en/products/detail/samsung-electro-m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
- C16: renamed from C22; PartNumber (none) -> CC0402JRNPO7BN220; PurchaseLink (none) -> https://www.digikey.de/en/products/detail/yageo/CC0402JRNPO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
- C17: renamed from C24; PartNumber (none) -> CC0603KRX7R7BB104; PurchaseLink (none) -> https://www.digikey.de/en/products/detail/yageo/CC0603KRX7R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
- C19: renamed from C25; PartNumber (none) -> CC0603KRX7R7BB104; PurchaseLink (none) -> https://www.digikey.de/en/products/detail/yageo/CC0603KRX7R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
- C21: renamed from C26; PartNumber (none) -> CL10A106MQ8NNNC; PurchaseLink (none) -> https://www.digikey.de/en/products/detail/samsung-electro-m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
- C25: renamed from C16; PartNumber (none) -> CC0603KRX7R7BB104; PurchaseLink (none) -> https://www.digikey.de/en/products/detail/yageo/CC0603KRX7R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
- C26: renamed from C17; PartNumber (none) -> CC0603KRX7R7BB104; PurchaseLink (none) -> https://www.digikey.de/en/products/detail/yageo/CC0603KRX7R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
- C27: renamed from C18; PartNumber (none) -> CC0603KRX7R7BB104; PurchaseLink (none) -> https://www.digikey.de/en/products/detail/yageo/CC0603KRX7R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
- C28: renamed from C19; PartNumber (none) -> CC0603KRX7R7BB104; PurchaseLink (none) -> https://www.digikey.de/en/products/detail/yageo/CC0603KRX7R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
- C29: renamed from C20; PartNumber (none) -> CL10A106MQ8NNNC; PurchaseLink (none) -> https://www.digikey.de/en/products/detail/samsung-electro-m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
- C33: renamed from C13; PartNumber (none) -> C0402C682K4RECAUTO; PurchaseLink (none) -> https://www.digikey.de/en/products/detail/kemet/C0402C682K4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
- C34: renamed from C15; PartNumber (none) -> C0603C103K4RECTU; PurchaseLink (none) -> https://www.digikey.de/en/products/detail/kemet/C0603C103K4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
- C35: renamed from C12; PartNumber (none) -> C0603C103K4RECTU; PurchaseLink (none) -> https://www.digikey.de/en/products/detail/kemet/C0603C103K4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
- C37: renamed from C14; PartNumber (none) -> C0402C682K4RECAUTO; PurchaseLink (none) -> https://www.digikey.de/en/products/detail/kemet/C0402C682K4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
- FB1, FB2: PartNumber (none) -> MH1608-121Y; PurchaseLink (none) -> https://www.digikey.de/en/products/detail/bourns-inc/mh1608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
- IC1: NumPart (none) -> 1727-6018-2-ND; PartNumber (none) -> SN74AHC1G125DCKR; PurchaseLink (none) -> https://www.digikey.de/en/products/detail/texas-instruments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
- R12: renamed from R26; PartNumber RC0603FR-071KL -> CRGP0603F470R; PurchaseLink https://www.digikey.com/en/products/detail/yageo/RC0603FR-0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 -> https://www.digikey.de/en/products/detail/te-connectivity-p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
- R13: renamed from R28; PartNumber RC0603FR-071KL -> CRGP0603F470R; PurchaseLink https://www.digikey.com/en/products/detail/yageo/RC0603FR-0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 -> https://www.digikey.de/en/products/detail/te-connectivity-p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
- R14: renamed from R29; PartNumber RC0603FR-071KL -> CRGP0603F470R; PurchaseLink https://www.digikey.com/en/products/detail/yageo/RC0603FR-0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 -> https://www.digikey.de/en/products/detail/te-connectivity-p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
- R15: renamed from R22; PartNumber (none) -> RCS06031M00FKEA; PurchaseLink (none) -> https://www.digikey.de/en/products/detail/vishay-dale/RCS06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
- R16: renamed from R20; PartNumber (none) -> RCS060310K0JNEA; PurchaseLink (none) -> https://www.digikey.de/en/products/detail/vishay-dale/RCS06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
- R18: renamed from R21; PartNumber (none) -> RCS060310K0JNEA; PurchaseLink (none) -> https://www.digikey.de/en/products/detail/vishay-dale/RCS06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
- R19: renamed from R24; PartNumber (none) -> CRGP0603F470R; PurchaseLink (none) -> https://www.digikey.de/en/products/detail/te-connectivity-p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
- R21: renamed from R25; PartNumber (none) -> CRGP0603F470R; PurchaseLink (none) -> https://www.digikey.de/en/products/detail/te-connectivity-p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
- R23: renamed from R14; PartNumber (none) -> RCS060310K0JNEA; PurchaseLink (none) -> https://www.digikey.de/en/products/detail/vishay-dale/RCS06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
- R25: renamed from R15; PartNumber (none) -> RCS060310K0JNEA; PurchaseLink (none) -> https://www.digikey.de/en/products/detail/vishay-dale/RCS06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
- R26: renamed from R16; PartNumber (none) -> RCS060310K0JNEA; PurchaseLink (none) -> https://www.digikey.de/en/products/detail/vishay-dale/RCS06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
- R27: renamed from R17; PartNumber (none) -> RCS060310K0JNEA; PurchaseLink (none) -> https://www.digikey.de/en/products/detail/vishay-dale/RCS06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
- R32: renamed from R23; PartNumber (none) -> RCS060312K4FKEA; PurchaseLink (none) -> https://www.digikey.de/en/products/detail/vishay-dale/RCS06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
- R39: renamed from R11; PartNumber (none) -> RCS060349R9FKEA; PurchaseLink (none) -> https://www.digikey.de/en/products/detail/vishay-dale/RCS06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
- R40: renamed from R18; PartNumber (none) -> RCS060349R9FKEA; PurchaseLink (none) -> https://www.digikey.de/en/products/detail/vishay-dale/RCS06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
- R41: renamed from R12; PartNumber (none) -> RCS060349R9FKEA; PurchaseLink (none) -> https://www.digikey.de/en/products/detail/vishay-dale/RCS06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
- R42: renamed from R19; PartNumber (none) -> RCS060349R9FKEA; PurchaseLink (none) -> https://www.digikey.de/en/products/detail/vishay-dale/RCS06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
- R43: renamed from R13; PartNumber (none) -> RCS060310R0FKEA; PurchaseLink (none) -> https://www.digikey.de/en/products/detail/vishay-dale/RCS06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
- SJ1, SJ2, SJ3: symbol ArchiBot-eagle-import:SOLDERJUMPERREFLOW_NOPASTE -> Jumper:SolderJumper_2_Open; now left out of the parts list
- U$1: PartNumber (none) -> W5500; PurchaseLink (none) -> https://www.digikey.de/en/products/detail/wiznet/W5500/4425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
- Y1: NumPart (none) -> 3305-3225S42500BMDAODGEE-TR-ND; PartNumber (none) -> 3305-3225S42500BMDAODGEE-TR-ND; PurchaseLink (none) -> https://www.digikey.de/en/products/detail/hkc/3225S42500BMD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
- renumbered D11 to D7, D13 to D8, D14 to D9
Connections:
- net +3V3: now also X1.10 (VC-), X1.12 (LED2_A)
- net AGND: no longer C19.2
- net GND: now also C19.2, C30.1 (C), C31.1 (C), C32.2, C36.1 (C), C39.1, C40.2, C41.1 (C), L2.7, L2.8, R45.1, U5.3 (ANODE), X1. (Shield)
- net GREENLED: now also X1.9 (VC+)
- net RX+: now also R34.2; no longer U$1.6 (RXP)
- net RX-: now also R33.2; no longer U$1.5 (RXN)
- net TX+: now also R31.2, X1.5 (TX+); no longer U$1.2 (TXP)
- net TX-: now also R30.2, X1.6 (TX-); no longer U$1.1 (TXN)
- net YELLOWLED: now also X1.11 (LED2_K)
- net at C33.1: now also X1.1 (RX+)
- net at C34.1, R40.1, R42.1: now also X1.3 (RCT)
- net at C35.1, R43.1: now also X1.4 (TCT)
- net at C37.1: now also X1.2 (RX-)
- new net: R29.1, U3.2 (L)
- new net: R37.1, U4.1
- new net: C30.2 (A), C31.2 (A), D13.2 (K), L3.1, R37.2, R38.2
- new net: C24.1, D12.1 (K), U4.4
- new net: D12.2 (A), R36.2
- new net: C38.2, R44.1, R45.2, U5.2 (REF)
- new net: C18.1, C20.1, C22.1, C23.1 (C), C24.2, D11.1 (A), L2.1, Q1.3 (D), R28.1, U3.4 (S)
- new net: C22.2, R35.2, U3.1 (C), U3.5 (F), U4.3
- new net: R30.1, U$1.1 (TXN)
- new net: R24.1, R28.2, U3.3 (X)
- new net: C20.2, D11.2 (K), L2.4, U3.7 (D)
- new net: D10.1 (A), Q1.1 (G), R20.2
- new net: D13.1 (A), L2.10, L2.9
- new net: L2.2, R36.1
- new net: D10.2 (K), R22.1
- new net: C32.1, C38.1, R38.1, U4.2, U5.1 (CATHODE)
- new net: C23.2 (A), R35.1
- new net: R34.1, U$1.6 (RXP)
- new net: R33.1, U$1.5 (RXN)
- new net: R31.1, U$1.2 (TXP)
- new net VBAT: C36.2 (A), C39.2, C40.1, C41.2 (A), L3.2, R44.2
- new net VC1: C13.2, C18.2, L2.3, R17.2, R22.2, R24.2, R29.2, X1.9 (VC+)
- new net VC2: C13.1, Q1.2 (S), R17.1, R20.1, X1.10 (VC-)
Other:
- note added: "10mAac"
- note added: "150mAdc"
- note added: "2Adc"
- note added: "30Vac"
- note added: "5Vdc"
- note added: "60Vdc"
- note added: "Circuit POE"
- note removed: "array x2"
- moved on the sheet: C14, C15, C16, C17, C19, C21, C25, C26, C27, C28, C29, D7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

Commit message: Add files via upload
Parts:
- C13: footprint CAP-1808 -> Capacitor_SMD:C_1812_4532Metric_Pad1.57x3.40mm_HandSolder; PartNumber GRM21BR61H106KE43K -> 18125G106ZAT2A; PurchaseLink https://www.digikey.de/en/products/detail/murata-electronic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 -> https://www.digikey.de/en/products/detail/kyocera-avx/18125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
- C18, C24: footprint CAP-0805 -> Capacitor_SMD:C_1206_3216Metric; PartNumber CL21B105KBFNNNG -> CL31B105KBHNNNE; PurchaseLink https://www.digikey.de/en/products/detail/samsung-electro-mechanics/CL21B105KBFNNNG/3894467 -> https://www.digikey.de/en/products/detail/samsung-electro-mechanics/CL31B105KBHNNNE/3886726
- C20: footprint CAP-0805 -> Capacitor_SMD:C_1206_3216Metric; PartNumber CL10C470JC81PNC -> CC1206JRNPO0BN470; PurchaseLink https://www.digikey.de/en/products/detail/samsung-electro-m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 -> https://www.digikey.de/en/products/detail/yageo/CC1206JRNPO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
- C22: footprint CAP-0805 -> Capacitor_SMD:C_1206_3216Metric; PartNumber CC0603ZRY5V9BB104 -> 1206B104K500CT; PurchaseLink https://www.digikey.de/en/products/detail/yageo/CC0603ZRY5V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 -> https://www.digikey.de/en/products/detail/walsin-technology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
- C23: footprint C3216TT(A) -> Capacitor_SMD:C_0805_2012Metric; CAPACITANCE 10uF -> (none); CASE CODE (IMPERIAL) 1206 -> (none); CASE CODE (METRIC) 3216 -> (none); CASE/PACKAGE 1206 -> (none); CONSTRUCTION Flat -> (none); DEPTH 1.6mm -> (none); DIELECTRIC MATERIAL Tantalum -> (none); DISSIPATION FACTOR 6% -> (none); ESR (EQUIVALENT SERIES RESISTANCE) 4R -> (none); FEATURES General Purpose -> (none); HEIGHT 1.6mm -> (none); HEIGHT - SEATED (MAX) 0.071inch -> (none); LEAD FREE Lead Free -> (none); LEAD PITCH 1.2mm -> (none); LEAKAGE CURRENT 1uA -> (none); LENGTH 3.2mm -> (none); LIFE (HOURS) 2000Hour -> (none); MAX OPERATING TEMPERATURE 125°C -> (none); MIN OPERATING TEMPERATURE -55°C -> (none); MOUNT Surface Mount -> (none); NUMBER OF PINS 2 -> (none); PACKAGE QUANTITY 2000 -> (none); PACKAGING Tape and Reel -> (none); POLARITY Polar -> (none); PurchaseLink https://www.digikey.de/en/products/detail/murata-electronic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 -> https://www.digikey.de/en/products/detail/samsung-electro-m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; RADIATION HARDENING No -> (none); REACH SVHC No SVHC -> (none); ROHS COMPLIANT Yes -> (none); SERIES T491 -> (none); SIZE 1.6mm -> (none); TERMINATION SMD/SMT -> (none); TOLERANCE 20% -> (none); VOLTAGE 10V -> (none); VOLTAGE RATING 10V -> (none); VOLTAGE RATING (DC) 10V -> (none); WEIGHT 0.000571oz -> (none); WIDTH 0.063inch -> (none)
- C30: footprint C6032TT(C) -> DatLibrery:22uF - 10V
- C31: footprint C3216TT(A) -> DatLibrery:10Uf 10v
- C32: footprint CAP-0603 -> DatLibrery:0.33 50v; PartNumber TAJA334K050RNJ -> C1608X7R1H334K080AC; PurchaseLink https://www.digikey.de/en/products/detail/kyocera-avx/TAJA3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 -> https://www.digikey.de/en/products/detail/tdk-corporation/C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
- C36: footprint C3216TT(A) -> DatLibrery:CAP330uF6V
- C38: footprint CAP-0603 -> Capacitor_SMD:C_0603_1608Metric
- C39: footprint CAP-0603 -> DatLibrery:10Uf 10v
- C40: footprint CAP-1808 -> DatLibrery:10uF-50V
- C41: footprint CAP-8.3EC -> DatLibrery:CAP-470uF16V
- D10: footprint DO-214AC/SMA -> DatLibrery:SMAJ12
- D11: footprint DO-214AC/SMA -> DatLibrery:NCSMAJ150A
- D12: footprint SOD-123(1-C,2-A) -> DatLibrery:BAV19
- D13: footprint DO-214AB/SMC -> DatLibrery:RBR5L40A
- L2: footprint SM13117EL -> DatLibrery:SM13117EL
- L3: footprint IND-0805 -> DatLibrery:IND-0805
- Q1, U5: footprint SOT23-3L -> DatLibrery:SOT23-3L
- R17: footprint Resistor_SMD:R_0603_1608Metric -> Capacitor_SMD:C_1206_3216Metric; PurchaseLink https://www.digikey.de/en/products/detail/vishay-dale/RCS06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 -> https://www.digikey.de/en/products/detail/stackpole-electro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
- R20: footprint Resistor_SMD:R_0603_1608Metric -> Capacitor_SMD:C_1206_3216Metric; PartNumber RCS060315K0FKEA -> RMCF1206FT15K0; PurchaseLink https://www.digikey.de/en/products/detail/vishay-dale/RCS06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 -> https://www.digikey.de/en/products/detail/stackpole-electro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
- R22: footprint Resistor_SMD:R_0603_1608Metric -> Capacitor_SMD:C_1206_3216Metric; PartNumber RCS060351K0FKEA -> RC1206FR-0751K1L; PurchaseLink https://www.digikey.de/en/products/detail/vishay-dale/RCS06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 -> https://www.digikey.de/en/products/detail/yageo/RC1206FR-07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
- R24: footprint Resistor_SMD:R_0603_1608Metric -> Capacitor_SMD:C_0805_2012Metric; PurchaseLink https://www.digikey.de/en/products/detail/vishay-dale/RCS06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 -> https://www.digikey.de/en/products/detail/koa-speer-electro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
- R28: footprint Resistor_SMD:R_0603_1608Metric -> Resistor_SMD:R_1206_3216Metric
- R29: footprint Resistor_SMD:R_0603_1608Metric -> Resistor_SMD:R_0805_2012Metric; PartNumber RCS0603680KFKEA -> RK73B2ATTD684J; PurchaseLink https://www.digikey.de/en/products/detail/vishay-dale/RCS06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 -> https://www.digikey.de/en/products/detail/koa-speer-electro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
- R35: footprint Resistor_SMD:R_0603_1608Metric -> Capacitor_SMD:C_1206_3216Metric; PartNumber RCS06035R10FKEA -> M251206BB5108JP500; PurchaseLink https://www.digikey.de/en/products/detail/vishay-dale/RCS06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 -> https://www.digikey.de/en/products/detail/vishay-beyschlag-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
- R36: footprint Resistor_SMD:R_0603_1608Metric -> Capacitor_SMD:C_1206_3216Metric; PartNumber RCS0603100RFKEA -> Y1630100R000Q9R; PurchaseLink https://www.digikey.de/en/products/detail/vishay-dale/RCS06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 -> https://www.digikey.de/en/products/detail/vpg-foil-resistor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
- R37: footprint Resistor_SMD:R_0603_1608Metric -> Capacitor_SMD:C_1206_3216Metric; PartNumber RCS060375R0FKEA -> RMCF1206FT75R0; PurchaseLink https://www.digikey.de/en/products/detail/vishay-dale/RCS06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 -> https://www.digikey.de/en/products/detail/stackpole-electro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
- R38: footprint Resistor_SMD:R_0603_1608Metric -> Capacitor_SMD:C_1206_3216Metric; PartNumber RCS06031K00FKEA -> RC1206FR-071KL; PurchaseLink https://www.digikey.de/en/products/detail/vishay-dale/RCS06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 -> https://www.digikey.de/en/products/detail/yageo/RC1206FR-07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
- U3: footprint DIP-08 -> DatLibrery:DIP-08
- U4: footprint PC357 -> DatLibrery:PC357
Other:
- moved on the sheet: C24, R17, R28

Commit message: Add files via upload
Parts:
- C36: CAPACITANCE 10uF -> (none); CASE CODE (IMPERIAL) 1206 -> (none); CASE CODE (METRIC) 3216 -> (none); CASE/PACKAGE 1206 -> (none); CONSTRUCTION Flat -> (none); DEPTH 1.6mm -> (none); DIELECTRIC MATERIAL Tantalum -> (none); DISSIPATION FACTOR 6% -> (none); ESR (EQUIVALENT SERIES RESISTANCE) 4R -> (none); FEATURES General Purpose -> (none); HEIGHT 1.6mm -> (none); HEIGHT - SEATED (MAX) 0.071inch -> (none); LEAD FREE Lead Free -> (none); LEAD PITCH 1.2mm -> (none); LEAKAGE CURRENT 1uA -> (none); LENGTH 3.2mm -> (none); LIFE (HOURS) 2000Hour -> (none); MAX OPERATING TEMPERATURE 125°C -> (none); MIN OPERATING TEMPERATURE -55°C -> (none); MOUNT Surface Mount -> (none); NUMBER OF PINS 2 -> (none); PACKAGE QUANTITY 2000 -> (none); PACKAGING Tape and Reel -> (none); POLARITY Polar -> (none); RADIATION HARDENING No -> (none); REACH SVHC No SVHC -> (none); ROHS COMPLIANT Yes -> (none); SERIES T491 -> (none); SIZE 1.6mm -> (none); TERMINATION SMD/SMT -> (none); TOLERANCE 20% -> (none); VOLTAGE 10V -> (none); VOLTAGE RATING 10V -> (none); VOLTAGE RATING (DC) 10V -> (none); WEIGHT 0.000571oz -> (none); WIDTH 0.063inch -> (none)
- C41: CAPACITANCE 10uF -> (none); CASE CODE (IMPERIAL) 1206 -> (none); CASE CODE (METRIC) 3216 -> (none); CASE/PACKAGE 1206 -> (none); CONSTRUCTION Flat -> (none); DEPTH 1.6mm -> (none); DIELECTRIC MATERIAL Tantalum -> (none); DISSIPATION FACTOR 6% -> (none); ESR (EQUIVALENT SERIES RESISTANCE) 4R -> (none); FEATURES General Purpose -> (none); HEIGHT 1.6mm -> (none); HEIGHT - SEATED (MAX) 0.071inch -> (none); LEAD FREE Lead Free -> (none); LEAD PITCH 1.2mm -> (none); LEAKAGE CURRENT 1uA -> (none); LENGTH 3.2mm -> (none); LIFE (HOURS) 2000Hour -> (none); MAX OPERATING TEMPERATURE 125°C -> (none); MIN OPERATING TEMPERATURE -55°C -> (none); MOUNT Surface Mount -> (none); NUMBER OF PINS 2 -> (none); PACKAGE QUANTITY 2000 -> (none); PACKAGING Tape and Reel -> (none); POLARITY Polar -> (none); PartNumber CAP TANT 470UF 20% 20V 3226 -> PCG1C471MCL1GS; PurchaseLink https://www.digikey.de/en/products/detail/vishay-sprague/59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 -> https://www.digikey.com/en/products/detail/nichicon/PCG1C47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; RADIATION HARDENING No -> (none); REACH SVHC No SVHC -> (none); ROHS COMPLIANT Yes -> (none); SERIES T491 -> (none); SIZE 1.6mm -> (none); TERMINATION SMD/SMT -> (none); TOLERANCE 20% -> (none); VOLTAGE 10V -> (none); VOLTAGE RATING 10V -> (none); VOLTAGE RATING (DC) 10V -> (none); WEIGHT 0.000571oz -> (none); WIDTH 0.063inch -> (none)
- D10: LinkPart https://www.digikey.de/en/products/detail/taiwan-semiconduc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 -> (none); NumPart SMAJ12 -> (none)
- D13: LinkPart https://www.digikey.de/en/products/detail/rohm-semiconducto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 -> (none); NumPart RBR5L40ADDTE25 -> (none)
- IC1: footprint NSARCHI:74AHC1G125 -> anetLib:74AHC1G125
- L2: LinkPart https://www.digikey.de/en/products/detail/bourns-inc/SM1311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 -> (none); NumPart SM13117EL -> (none)
- Q1: LinkPart https://www.digikey.de/en/products/detail/diotec-semiconduc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 -> (none); NumPart 2N7002 -> (none)
- SJ1, SJ2, SJ3: footprint NSARCHI:SJ -> anetLib:Jumper
- U$1: footprint NSARCHI:W5500 -> anetLib:W5500
- U3: LinkPart https://www.digikey.de/de/products/detail/power-integration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 -> (none); NumPart DPA423GN-TL -> (none)
- U4: LinkPart https://www.digikey.de/en/products/detail/sharp-socle-techn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 -> (none); NumPart PC357N2J000F -> (none)
- U5: LinkPart Shunt Voltage Reference IC Adjustable 2.495V 36 VV ±2.2% 10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 -> (none); NumPart TL431ID -> (none)
- X1: footprint NSARCHI:RB1-125BAG1A -> anetLib:7499210121A; LinkPart https://www.digikey.de/en/products/detail/w%C3%BCrth-elektr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 -> (none); NumPart 7499210121A -> (none)
Other:
- note added: "V-2.0"
- note removed: "matriz x4"

Commit message: #V.1
Parts:
- R15: PurchaseLink https://www.digikey.de/en/products/detail/vishay-dale/RCS06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 -> https://www.digikey.de/en/products/detail/koa-speer-electro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
- R38: PartNumber RC1206FR-071KL -> RCS06031K00FKEA; PurchaseLink https://www.digikey.de/en/products/detail/yageo/RC1206FR-07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 -> https://www.digikey.de/en/products/detail/vishay-dale/RCS06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
Changed lines of the file:
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@@
 			)
 		)
-		(property "PurchaseLink" "https://www.digikey.de/en/products/detail/vishay-dale/RCS06031M00FKEA/5866949"
+		(property "PurchaseLink" "https://www.digikey.de/en/products/detail/koa-speer-electronics-inc/RK73B2ATTD105J/10235908"
 			(at 112.395 120.015 0)
 			(effects
@@
 			)
 		)
-		(property "PartNumber" "RC1206FR-071KL"
+		(property "PartNumber" "RCS06031K00FKEA"
 			(at 283.21 333.375 0)
 			(effects
@@
 			)
 		)
-		(property "PurchaseLink" "https://www.digikey.de/en/products/detail/yageo/RC1206FR-071KL/728387"
+		(property "PurchaseLink" "https://www.digikey.de/en/products/detail/vishay-dale/RCS06035K10FKEA/5868559"
 			(at 283.21 333.375 0)
 			(effects
