File: Hardware/A-NET/MCU-WiFi.kicad_sch (KiCad schematic)
At the start: 26 parts, among them J2 USB_C_Receptacle_USB2.0_16P, SW1 SW_MEC_5E, SW2 SW_MEC_5E, U2 ESP32-S3-WROOM-1, U3 AMS1117-3.3

Commit message: add digikey | add POE
Parts:
- removed C10, C11, C8: 10uF, Capacitor_SMD:C_0603_1608Metric, symbol Device:C
- removed C9: 0.1uF, Capacitor_SMD:C_0603_1608Metric, symbol Device:C
- removed D10: LEDUSB, LED_SMD:LED_0603_1608Metric_Pad1.05x0.95mm_HandSolder, symbol Device:LED_Small_Filled
- removed R10: 75, Resistor_SMD:R_0603_1608Metric_Pad0.98x0.95mm_HandSolder, symbol Device:R
- removed U3: AMS1117-3.3, Package_TO_SOT_SMD:SOT-223-3_TabPin2, symbol Regulator_Linear:AMS1117-3.3
- C10: renamed from C7; PartNumber (none) -> CL10A106MQ8NNNC; PurchaseLink (none) -> https://www.digikey.de/en/products/detail/samsung-electro-m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
- C11: renamed from C29; PartNumber (none) -> CL10A106MQ8NNNC; PurchaseLink (none) -> https://www.digikey.de/en/products/detail/samsung-electro-m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
- C12: renamed from C28; PartNumber (none) -> CL10A106MQ8NNNC; PurchaseLink (none) -> https://www.digikey.de/en/products/detail/samsung-electro-m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
- C7: renamed from C30; PartNumber (none) -> CL10A106MQ8NNNC; PurchaseLink (none) -> https://www.digikey.de/en/products/detail/samsung-electro-m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
- C8: renamed from C31; PartNumber (none) -> CC0603KRX7R7BB104; PurchaseLink (none) -> https://www.digikey.de/en/products/detail/yageo/CC0603KRX7R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
- C9: renamed from C32; PartNumber (none) -> CL10A106MQ8NNNC; PurchaseLink (none) -> https://www.digikey.de/en/products/detail/samsung-electro-m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
- D6: PartNumber (none) -> 1N5819HW-7-F; PurchaseLink (none) -> https://www.digikey.de/en/products/detail/diodes-incorporat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
- J2: NumPart (none) -> 5622-44116B01231TR-ND; PartNumber (none) -> USB4105-GF-A; PurchaseLink (none) -> https://www.digikey.de/en/products/detail/gct/USB4105-GF-A/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
- R10: renamed from R32; PartNumber RC0603FR-071KL -> RCS06031K00FKEA; PurchaseLink https://www.digikey.com/en/products/detail/yageo/RC0603FR-0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 -> https://www.digikey.de/en/products/detail/vishay-dale/RCS06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
- R11: renamed from R31; PartNumber RC0603FR-071KL -> RCS06031K00FKEA; PurchaseLink https://www.digikey.com/en/products/detail/yageo/RC0603FR-0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 -> https://www.digikey.de/en/products/detail/vishay-dale/RCS06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
- R7: renamed from R33; PartNumber RC0603FR-071KL -> RCS06031K00FKEA; PurchaseLink https://www.digikey.com/en/products/detail/yageo/RC0603FR-0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 -> https://www.digikey.de/en/products/detail/vishay-dale/RCS06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
- R8: footprint Resistor_SMD:R_0201_0603Metric -> (none); LinkPart (none) -> https://www.digikey.de/en/products/detail/yageo/RC0603FR-07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; NumPart (none) -> RC0603FR-075K1L; PartNumber (none) -> RCS06035K10FKEA; PurchaseLink (none) -> https://www.digikey.de/en/products/detail/vishay-dale/RCS06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
- R9: LinkPart (none) -> https://docs.wiznet.io/img/osh/WIZnet_Pico_PoE/Sch_WIZnet_P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; NumPart (none) -> RC0603FR-075K1L; PartNumber (none) -> RCS06035K10FKEA; PurchaseLink (none) -> https://www.digikey.de/en/products/detail/vishay-dale/RCS06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
- SW1: renamed from SW2; LinkPart (none) -> https://www.digikey.com/en/products/detail/c-k/PTS645SM43SM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; NumPart (none) -> PTS645SM43SMTR92 LFS; PartNumber (none) -> PTS645SM43SMTR92 LFS; PurchaseLink (none) -> https://www.digikey.com/en/products/detail/c-k/PTS645SM43SM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
- SW2: renamed from SW1; LinkPart (none) -> https://www.digikey.com/en/products/detail/c-k/PTS645SM43SM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; NumPart (none) -> PTS645SM43SMTR92 LFS; PartNumber (none) -> PTS645SM43SMTR92 LFS; PurchaseLink (none) -> https://www.digikey.com/en/products/detail/c-k/PTS645SM43SM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
- U2: NumPart (none) -> 1965-ESP32-S3-WROOM-1-N8DKR-ND; PartNumber (none) -> ESP32-S3-WROOM-1-N8; PurchaseLink (none) -> https://www.digikey.de/en/products/detail/espressif-systems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
- renumbered D7 to D3, D8 to D4, D9 to D5
Connections:
- net +3V3USB renamed +3V3
- net Vout renamed VBAT
- no-connect marks 28 -> 30
Other:
- note added: "1K ,10K,1nF Cambiar 0805"
- note added: "5K1,10uF,1uF 0603 Button"
- note added: "En el lab:"
- note removed: "Regulador USB"
- moved on the sheet: C11, C12, R10, R11, SW1, SW2

Commit message: Add files via upload
Parts:
- U2: NumPart 1965-ESP32-S3-WROOM-1-N8DKR-ND -> (none)
Changed lines of the file:
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@@
 			)
 		)
-		(property "Datasheet" "https://www.vishay.com/docs/20065/rcse3.pdf"
+		(property "Datasheet" "https://www.digikey.de/en/supplier-centers/yageo"
 			(at 31.75 40.64 0)
 			(effects
@@
 			)
 		)
-		(property "Datasheet" "https://www.vishay.com/docs/20065/rcse3.pdf"
+		(property "Datasheet" "https://www.digikey.de/en/supplier-centers/yageo"
 			(at 269.875 51.435 0)
 			(effects
@@
 		)
 		(property "Description" "WiFi 802.11a/b/g/n, Bluetooth v5.0 Transceiver Module 2.4GHz PCB Trace"
-			(at 58.42 86.36 0)
-			(effects
-				(font
-					(size 1.27 1.27)
-				)
-				(hide yes)
-			)
-		)
-		(property "NumPart" "1965-ESP32-S3-WROOM-1-N8DKR-ND"
 			(at 58.42 86.36 0)
 			(effects
@@
 			)
 		)
-		(property "Datasheet" "https://www.vishay.com/docs/20065/rcse3.pdf"
+		(property "Datasheet" "https://www.digikey.de/en/supplier-centers/yageo"
 			(at 229.235 50.165 0)
 			(effects

Commit message: #V.1
Parts:
- R10, R11, R7: PurchaseLink https://www.digikey.de/en/products/detail/vishay-dale/RCS06031K00FKEA/5866934 -> https://www.digikey.de/en/products/detail/vishay-dale/RCS06035K10FKEA/5868559
Changed lines of the file:
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@@
 			)
 		)
-		(property "PurchaseLink" "https://www.digikey.de/en/products/detail/vishay-dale/RCS06031K00FKEA/5866934"
+		(property "PurchaseLink" "https://www.digikey.de/en/products/detail/vishay-dale/RCS06035K10FKEA/5868559"
 			(at 31.75 40.64 0)
 			(effects
@@
 			)
 		)
-		(property "PurchaseLink" "https://www.digikey.de/en/products/detail/vishay-dale/RCS06031K00FKEA/5866934"
+		(property "PurchaseLink" "https://www.digikey.de/en/products/detail/vishay-dale/RCS06035K10FKEA/5868559"
 			(at 269.875 51.435 0)
 			(effects
@@
 			)
 		)
-		(property "PurchaseLink" "https://www.digikey.de/en/products/detail/vishay-dale/RCS06031K00FKEA/5866934"
+		(property "PurchaseLink" "https://www.digikey.de/en/products/detail/vishay-dale/RCS06035K10FKEA/5868559"
 			(at 229.235 50.165 0)
 			(effects
