File: Hardware/A-NET.kicad_pcb (KiCad board)
At the start: 2 copper layers, 100 x 60 mm, 106 parts, among them IC1 74AHC1G125, J1 BAT, J2 USB_C_Receptacle_USB2.0_16P, J3 RJ45, J4 Power, J5 Analog, J6 Digital/PWM, J7 Digital/PWM, U1 TPS563252DRLR, U2 ESP32-S3-WROOM-1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

Commit message: .agregado modificaciones pcb
Parts:
- R12, R13, R14: moved to F.Cu
- R2: value 32K -> 47K
- moved D3 20.5 mm to (161.9, 86.8), turned to 180 degrees
- moved D7 14.6 mm to (170.4, 101.4)
- moved D6 12.4 mm to (172.5, 101.4), turned to 180 degrees
- moved C8 11.0 mm to (168.9, 87.9), turned to 90 degrees
- moved C9 8.73 mm to (170.5, 87.9), turned to 90 degrees
- moved D8 7.50 mm to (182.7, 89.1)
- moved D2 5.60 mm to (179.3, 85.0), turned to 0 degrees
- moved C6 5.58 mm to (173.0, 87.1), turned to 0 degrees
- moved C5 5.38 mm to (173.0, 88.7), turned to 0 degrees
- moved D4 4.82 mm to (171.1, 92.7), turned to -90 degrees
- moved C10 4.32 mm to (179.2, 81.2), turned to 0 degrees
- moved C1 4.10 mm to (179.1, 79.6)
- moved C7 3.05 mm to (190.8, 122.9), turned to 180 degrees
- moved R6 2.97 mm to (172.8, 92.7), turned to -90 degrees
- moved R12 2.96 mm to (141.0, 118.5)
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Connections:
- net /Ethernet/INTN renamed /Archi/INTN
- net /Ethernet/MISO renamed /Ethernet/MISO_MCU
- net /Ethernet/MOSI renamed /Archi/MOSI
- net /Ethernet/RESET renamed /Archi/RSTN
- net /Ethernet/SCK renamed /Archi/CLK
- C11 pad 1: /MCU-WiFi/CHIP_PU -> +3V3
- C11 pad 2: GND -> /MCU-WiFi/CHIP_PU
- C12 pad 1: /MCU-WiFi/GPIO0 -> +3V3
- C12 pad 2: GND -> /Archi/RESET_MCU
- J6 pad 5: /MCU-WiFi/GPIO0 -> /Archi/RESET_MCU
- R11 pad 1: /MCU-WiFi/GPIO0 -> /Archi/RESET_MCU
- U2 pad 27: /MCU-WiFi/GPIO0 -> /Archi/RESET_MCU
- U4 pad 2: /MCU-WiFi/GPIO0 -> /Archi/RESET_MCU
- U5 pad 1: /Archi/RUN -> GND
- U5 pad 2: GND -> /Archi/RUN
Routing:
- net /Archi/RESET_MCU: track 0.00 -> 42.6 mm
- net /MCU-WiFi/GPIO0: track 40.7 -> 0.00 mm
- net GND: track 49.8 -> 31.2 mm, vias 6 -> 8
- net Net-(SJ1-A): track 45.3 -> 30.0 mm
- net VBAT: track 27.9 -> 16.8 mm
- net +5VIN: track 74.9 -> 80.9 mm, vias 2 -> 0
- net /Ethernet/LINKLED: track 46.0 -> 40.4 mm, vias 3 -> 2
- net /MCU-WiFi/CHIP_PU: track 57.8 -> 53.7 mm
- net Net-(D1-A): track 13.1 -> 9.19 mm, vias 1 -> 0
- net /MCU-WiFi/D+: track 28.1 -> 24.2 mm, vias 2 -> 0
- net /Ethernet/ACTLED: track 40.1 -> 36.6 mm
- net /MCU-WiFi/D-: track 24.8 -> 22.1 mm, vias 2 -> 0
- net /Archi/GPIO2: track 109.0 -> 106.5 mm
- net /Archi/GPIO3: track 115.7 -> 113.3 mm
- net /Ethernet/DUPLED: track 6.84 -> 4.45 mm, vias 1 -> 0
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Other:
- board text added: "BOOT"
- board text added: "BOOTSEL"
- board text added: "ESP32-S3"
- board text added: "I/O ANALOGIC"
- board text added: "I/O DIGITAL"
- board text added: "Operation mode select pins"
- board text added: "RST"
