File: Hardware/Alimentación.kicad_sch (KiCad schematic)
At the start: 19 parts, among them J1 BAT, U1 TPS563252DRLR

Commit message: .agregado modificaciones pcb
Parts:
- R2: value 32K -> 47K
- R5: PartNumber RCS0603220KFKEA -> RT0603BRD07135KL; PurchaseLink https://www.digikey.com/en/products/detail/vishay-dale/RCS0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 -> https://www.digikey.com/en/products/detail/yageo/RT0603BRD0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
Other:
- title: (none) -> ArchiNET

Commit message: .add digikey
Parts:
- C3, C6: value 100nF -> 0.1uF
- R3: PartNumber RCS060310K0JNEA -> RCS060330K0FKEA; PurchaseLink https://www.digikey.com/en/products/detail/vishay-dale/RCS060310K0JNEA/5866963?s=N4IgTCBcDaIKwBYCMBaMAOJB2FqByAIiALoC%2BQA -> https://www.digikey.com/en/products/detail/vishay-dale/RCS060330K0FKEA/5868642
Changed lines of the file:
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@@
 			)
 		)
-		(property "Description" "Unpolarized capacitor, small symbol"
+		(property "Description" "CAP CER 22UF 10V X5R 0603"
 			(at 335.28 73.66 0)
 			(effects
@@
 			)
 		)
-		(property "Value" "100nF"
+		(property "Value" "0.1uF"
 			(at 276.098 75.184 0)
 			(effects
@@
 			)
 		)
-		(property "Description" "Unpolarized capacitor, small symbol"
+		(property "Description" "CAP CER 0.1UF 16V X7R 0603"
 			(at 275.59 73.66 0)
 			(effects
@@
 			)
 		)
-		(property "Value" "100nF"
+		(property "Value" "0.1uF"
 			(at 342.138 75.184 0)
 			(effects
@@
 			)
 		)
-		(property "Description" "Unpolarized capacitor, small symbol"
+		(property "Description" "CAP CER 0.1UF 16V X7R 0603"
 			(at 341.63 73.66 0)
 			(effects
@@
 			)
 		)
-		(property "Description" "Unpolarized capacitor, small symbol"
+		(property "Description" "CAP CER 56PF 25V X8R 0603"
 			(at 327.66 80.01 0)
 			(effects
@@
 			)
 		)
-		(property "Description" ""
+		(property "Description" "IC REG BUCK ADJ 3A SOT563"
 			(at 297.18 71.12 0)
 			(effects
@@
 			)
 		)
-		(property "Description" "Unpolarized capacitor, small symbol"
+		(property "Description" "CAP CER 10UF 16V X6S 0603"
 			(at 262.89 73.66 0)
 			(effects
@@
 			)
 		)
-		(property "Description" "Inductor"
+		(property "Description" "FIXED IND 2.2UH 4.3A 48 MOHM SMD"
 			(at 323.85 66.04 0)
 			(effects
@@
 			)
 		)
-		(property "Description" "Unpolarized capacitor, small symbol"
+		(property "Description" "CAP CER 10UF 16V X6S 0603"
 			(at 269.24 73.66 0)
 			(effects
@@
 			)
 		)
-		(property "PartNumber" "RCS060310K0JNEA"
+		(property "PartNumber" "RCS060330K0FKEA"
 			(at 320.04 78.74 0)
 			(effects
@@
 			)
 		)
-		(property "PurchaseLink" "https://www.digikey.com/en/products/detail/vishay-dale/RCS060310K0JNEA/5866963?s=N4IgTCBcDaIKwBYCMBaMAOJB2FqByAIiALoC%2BQA"
+		(property "PurchaseLink" "https://www.digikey.com/en/products/detail/vishay-dale/RCS060330K0FKEA/5868642"
 			(at 320.04 78.74 0)
 			(effects
