File: Hardware/Archi.kicad_sch (KiCad schematic)
At the start: 19 parts, among them J4 Power, J5 Analog, J6 Digital/PWM, J7 Digital/PWM, U5 SWITCH

Commit message: .add modificaciónes
Connections:
- net MISO renamed MISO/TX
- net MOSI renamed MOSI/RX
Other:
- moved on the sheet: A0, A1, A2, A3
