File: Hardware/MCU-WiFi.kicad_sch (KiCad schematic)
At the start: 19 parts, among them J2 USB_C_Receptacle_USB2.0_16P, U2 ESP32-S3-WROOM-1, U3 SWITCH, U4 SWITCH

Commit message: .agregado modificaciones pcb
Parts:
- R8, R9: LinkPart https://www.digikey.com/en/products/detail/panasonic-electr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 -> (none); NumPart ERJ-PA2F5101X -> (none)
- U3, U4: symbol anetLib:PTS645SM43SMTR92LFS -> Switch:SW_Push_Dual_x2
Connections:
- net +3V3: now also C11.1, C12.1
- net CHIP_PU: now also C11.2; no longer C11.1, U3.4
- net GND: no longer C11.2, C12.2, U3.3, U4.3
- net RESET: now also C12.2; no longer C12.1, U4.4
Other:
- note added: "BOOT/RESET"
- title: (none) -> ArchiNET
- moved on the sheet: C11, R10, R11
