File: Hardware/A-NET.kicad_sch (KiCad schematic)
At the start: 0 parts

Commit message: .agregado modificaciones pcb
Other:
- sheet Ethernet ports: added MISO; removed MISO_MCU
- title: (none) -> ArchiNET

Commit message: .add modificaciónes
Other:
- sheet Archi ports: added MISO/TX, MOSI/RX; removed MISO, MOSI
- note added: "ARCHI"
- note added: "ESP32-S3"
- note added: "ETHERNET WIZNET W5500"
- note added: "FUENTE DE ALIMENTACIÓN"
Changed lines of the file:
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@@
+		)
+	)
+	(text "ESP32-S3"
+		(exclude_from_sim no)
+		(at 200.66 73.914 0)
+		(effects
+			(font
+				(size 2.54 2.54)
+				(thickness 0.508)
+				(bold yes)
+			)
+		)
+	)
+	(text "  ETHERNET\nWIZNET W5500"
+		(exclude_from_sim no)
+		(at 199.898 117.602 0)
+		(effects
+			(font
+				(size 2.032 2.032)
+				(thickness 0.508)
+				(bold yes)
+			)
 		)
 	)
@@
 		)
 	)
+	(text " FUENTE DE \nALIMENTACIÓN"
+		(exclude_from_sim no)
+		(at 96.52 71.628 0)
+		(effects
+			(font
+				(size 2.54 2.54)
+				(thickness 0.508)
+				(bold yes)
+			)
+		)
+	)
+	(text "ARCHI"
+		(exclude_from_sim no)
+		(at 143.002 75.692 0)
+		(effects
+			(font
+				(size 2.54 2.54)
+				(thickness 0.508)
+				(bold yes)
+			)
+		)
+	)
 	(junction
 		(at 166.37 66.04)
@@
 			)
 		)
-		(pin "MOSI" input
+		(pin "MOSI{slash}RX" input
 			(at 161.29 63.5 0)
 			(effects
@@
 			)
 		)
-		(pin "MISO" input
+		(pin "MISO{slash}TX" input
 			(at 161.29 66.04 0)
 			(effects
