File: Hardware/Ethernet.kicad_sch (KiCad schematic)
At the start: 45 parts, among them IC1 74AHC1G125, J3 RJ45, Y1 25MHz

Commit message: .agregado modificaciones pcb
Parts:
- IC1: NumPart 1727-6018-2-ND -> (none)
- Y1: NumPart 3305-3225S42500BMDAODGEE-TR-ND -> (none)
Connections:
- net MISO: now also IC1.4 (Y); no longer IC1.2 (A), U$1.34 (MISO)
- net MISO_MCU: now also IC1.2 (A), U$1.34 (MISO); no longer IC1.4 (Y)
Other:
- title: (none) -> ArchiNET

Commit message: .add digikey
Parts:
- SJ1, SJ2, SJ3: PartNumber (none) -> -; PurchaseLink (none) -> -
- Y1: PurchaseLink https://www.digikey.de/en/products/detail/hkc/3225S42500BMD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 -> https://www.digikey.com/en/products/detail/abracon-llc/ABM3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
Changed lines of the file:
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@@
 			)
 		)
-		(property "Description" ""
+		(property "Description" "Resistor, small symbol"
 			(at 80.645 118.11 0)
 			(effects
@@
 			)
 		)
-		(property "Description" ""
+		(property "Description" "CAP CER 0.1UF 16V X7R 0603"
 			(at 210.185 85.725 0)
 			(effects
@@
 			)
 		)
-		(property "Datasheet" "~"
+		(property "Datasheet" "-"
 			(at 125.095 67.31 0)
 			(effects
@@
 			)
 		)
+		(property "PartNumber" "-"
+			(at 125.095 67.31 0)
+			(effects
+				(font
+					(size 1.27 1.27)
+				)
+			)
+		)
+		(property "PurchaseLink" "-"
+			(at 125.095 67.31 0)
+			(effects
+				(font
+					(size 1.27 1.27)
+				)
+			)
+		)
 		(pin "2"
 		)
@@
 			)
 		)
-		(property "Datasheet" "~"
+		(property "Datasheet" "https://abracon.com/Resonators/abm3b.pdf"
 			(at 78.74 127 0)
 			(effects
@@
 			)
 		)
-		(property "PurchaseLink" "https://www.digikey.de/en/products/detail/hkc/3225S42500BMDAODGEE-TR/15292356?https://www.digikey.com/en/products/detail/abracon-llc/ABM3B-25-000MHZ-22-E-4-H-T/8582001"
+		(property "PurchaseLink" "https://www.digikey.com/en/products/detail/abracon-llc/ABM3B-25-000MHZ-22-E-4-H-T/8582001"
 			(at 78.74 127 0)
 			(effects
@@
 			)
 		)
-		(property "Description" ""
+		(property "Description" "Resistor, small symbol"
 			(at 104.14 148.59 0)
 			(effects
@@
 			)
 		)
-		(property "Description" ""
+		(property "Description" "CAP CER 6800PF 16V X7R 0603"
 			(at 323.215 69.85 0)
 			(effects
@@
 			)
 		)
-		(property "Description" ""
+		(property "Description" "Resistor, small symbol"
 			(at 89.535 95.25 0)
 			(effects
@@
 			)
 		)
-		(property "Description" ""
+		(property "Description" "Resistor, small symbol"
 			(at 156.21 64.643 0)
 			(effects
@@
 			)
 		)
-		(property "Datasheet" "~"
+		(property "Datasheet" "-"
 			(at 137.795 67.31 0)
 			(effects
@@
 			)
 		)
+		(property "PartNumber" "-"
+			(at 137.795 67.31 0)
+			(effects
+				(font
+					(size 1.27 1.27)
+				)
+			)
+		)
+		(property "PurchaseLink" "-"
+			(at 137.795 67.31 0)
+			(effects
+				(font
+					(size 1.27 1.27)
+				)
+			)
+		)
 		(pin "1"
 		)
@@
 			)
 		)
-		(property "Description" ""
+		(property "Description" "Resistor, small symbol"
 			(at 318.135 82.55 0)
 			(effects
@@
 			)
 		)
-		(property "Description" ""
+		(property "Description" "CAP CER 22PF 16V C0G/NP0 0603"
 			(at 69.85 133.35 0)
 			(effects
@@
 			)
 		)
-		(property "Datasheet" "~"
+		(property "Datasheet" "-"
 			(at 150.495 67.31 0)
 			(effects
@@
 			)
 		)
+		(property "PartNumber" "-"
+			(at 150.495 67.31 0)
+			(effects
+				(font
+					(size 1.27 1.27)
+				)
+			)
+		)
+		(property "PurchaseLink" "-"
+			(at 150.495 67.31 0)
+			(effects
+				(font
+					(size 1.27 1.27)
+				)
+			)
+		)
 		(pin "2"
 		)
@@
 			)
 		)
-		(property "Description" ""
+		(property "Description" "Resistor, small symbol"
 			(at 96.52 138.43 0)
 			(effects
@@
 			)
 		)
-		(property "Description" ""
+		(property "Description" "FERRITE BEAD 120 OHM 0603 1LN"
 			(at 201.93 51.435 0)
 			(effects
@@
 			)
 		)
-		(property "Description" ""
+		(property "Description" "CAP CER 0603 10NF 16V X7R 10%"
 			(at 302.895 71.12 0)
 			(effects
@@
 			)
 		)
-		(property "Description" ""
+		(property "Description" "Resistor, small symbol"
 			(at 320.675 54.61 0)
 			(effects
@@
 			)
 		)
-		(property "Description" ""
+		(property "Description" "FERRITE BEAD 120 OHM 0603 1LN"
 			(at 201.93 60.325 0)
 			(effects
@@
 			)
 		)
-		(property "Description" ""
+		(property "Description" "Resistor, small symbol"
 			(at 323.215 82.55 0)
 			(effects
@@
 			)
 		)
-		(property "Description" ""
+		(property "Description" "Resistor, small symbol"
 			(at 315.595 54.61 0)
 			(effects
@@
 			)
 		)
-		(property "Description" ""
+		(property "Description" "CAP CER 0.1UF 16V X7R 0603"
 			(at 90.805 161.29 0)
 			(effects
@@
 			)
 		)
-		(property "Description" ""
+		(property "Description" "Resistor, small symbol"
 			(at 325.755 54.61 0)
 			(effects
@@
 			)
 		)
-		(property "Description" ""
+		(property "Description" "Resistor, small symbol"
 			(at 143.002 64.643 0)
 			(effects
@@
 			)
 		)
-		(property "Description" ""
+		(property "Description" "CAP CER 6800PF 16V X7R 0603"
 			(at 333.375 74.93 0)
 			(effects
@@
 			)
 		)
-		(property "Description" ""
+		(property "Description" "CAP CER 10UF 16V X6S 0603"
 			(at 78.105 161.29 0)
 			(effects
@@
 			)
 		)
-		(property "Description" ""
+		(property "Description" "CAP CER 0.1UF 16V X7R 0603"
 			(at 202.565 85.725 0)
 			(effects
@@
 			)
 		)
-		(property "Description" ""
+		(property "Description" "CAP CER 0603 10NF 16V X7R 10%"
 			(at 323.215 97.79 0)
 			(effects
@@
 			)
 		)
-		(property "Description" ""
+		(property "Description" "CAP CER 10UF 16V X6S 0603"
 			(at 135.255 162.56 0)
 			(effects
@@
 			)
 		)
-		(property "Description" ""
+		(property "Description" "CAP CER 10UF 16V X6S 0603"
 			(at 233.045 85.725 0)
 			(effects
@@
 			)
 		)
-		(property "Description" ""
+		(property "Description" "Resistor, small symbol"
 			(at 180.975 125.73 0)
 			(effects
@@
 			)
 		)
-		(property "Description" "Resistor"
+		(property "Description" "Resistor, small symbol"
 			(at 115.824 64.643 0)
 			(effects
@@
 			)
 		)
-		(property "Description" ""
+		(property "Description" "CAP CER 0.1UF 16V X7R 0603"
 			(at 217.805 85.725 0)
 			(effects
@@
 			)
 		)
-		(property "Description" ""
+		(property "Description" "CAP CER 0.1UF 16V X7R 0603"
 			(at 225.425 85.725 0)
 			(effects
@@
 			)
 		)
-		(property "Description" ""
+		(property "Description" "Resistor, small symbol"
 			(at 95.885 95.25 0)
 			(effects
@@
 			)
 		)
-		(property "Description" ""
+		(property "Description" "Resistor, small symbol"
 			(at 130.048 64.897 0)
 			(effects
@@
 			)
 		)
-		(property "Description" ""
+		(property "Description" "CAP CER 0.1UF 16V X7R 0603"
 			(at 127.635 162.56 0)
 			(effects
@@
 			)
 		)
-		(property "Description" ""
+		(property "Description" "CAP CER 22PF 16V C0G/NP0 0603"
 			(at 86.36 133.35 0)
 			(effects

Commit message: .add modificaciónes
Parts:
- added TP2: CLKIN, TestPoint:TestPoint_THTPad_1.0x1.0mm_Drill0.5mm, symbol Connector:TestPoint
- added TP3: AVDD, TestPoint:TestPoint_THTPad_1.0x1.0mm_Drill0.5mm, symbol Connector:TestPoint
- added TP4: AGND, TestPoint:TestPoint_THTPad_1.0x1.0mm_Drill0.5mm, symbol Connector:TestPoint
Connections:
- net AGND: now also TP4.1
- net AVDD: now also TP3.1
- net at C15.1, R15.2, U$1.30 (XI/CLKIN)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: now also TP2.1
Other:
- moved on the sheet: C13, C15, C19, C20, C21, C22, C23, R15, Y1
